Commit message: Fix URDF laser frame mismatch, add relevance distance filter, document odom migration
1. robot.urdf: Rename LiDAR frame from "base_laser" to "laser" to match
   slam.launch.py, ld19.yaml, and the LiDAR driver's frame_id override.
   The mismatch caused a TF tree split when robot_state_publisher and
   slam.launch.py ran simultaneously — slam_toolbox couldn't resolve
   the scan frame because RSP published base_link→base_laser while the
   static TF published base_link→laser.

2. admin_node.py: Add cosine distance threshold filter (default 1.0) that
   discards irrelevant chunks BEFORE the LLM sees them.  Out-of-scope
   questions (e.g. "What is the capital of France?") are short-circuited
   with a canned response, saving a full Ollama inference round-trip
   (5-30s on Jetson).  Configurable via relevance_distance_threshold param.

3. dummy_odom.py: Document known map-shearing limitation and the 3-step
   migration path (rf2o → wheel encoders → IMU-fused EKF).

4. mecanum_driver_node.py: Document the future encoder odometry path in
   serial_reader — forward kinematics formulas and the steps needed when
   Arduino firmware adds encoder tick reporting.

Co-Authored-By: Claude Opus 4.6 <noreply@anthropic.com>

File: jetson/robot_description/urdf/robot.urdf (robot description, URDF)
Before this commit: robot my_robot, 3 links, 2 joints
Links:
- removed link base_laser
- added link laser
Joints:
- joint laser_joint: child base_laser -> laser
